File: pcb/h7_breakout.kicad_sch (KiCad schematic)
At the start: 68 parts, among them J1 USB_B, J10 RJ45_pyControl, J11 RJ45_pyControl, J12 RJ45_pyControl, J13 RJ45_pyControl, J14 RJ45_pyControl, J15 RJ45_pyControl, J16 Conn_01x06_Pin, J2 PJ-037A, J3 SWD_connector, J4 RJ45_pyControl, J5 RJ45_pyControl, J6 RJ45_pyControl, J7 RJ45_pyControl, J8 RJ45_pyControl, J9 RJ45_pyControl, U1 R-78E5.0-1.0, U10 SRV05-4, U11 SRV05-4, U12 SRV05-4, U13 SRV05-4, U14 SRV05-4, U15 SRV05-4, U16 SRV05-4, U17 SRV05-4, U18 SRV05-4, U19 SRV05-4, U2 AMS1117-3.3, U20 SRV05-4, U3 USBLC6-2SC6, U4 STM32H743VIT6, U5 W25Q25PWSSIQ, U6 TBD62083APG, U7 TBD62083APG, U8 TBD62083APG, U9 SRV05-4, Y1 25 MHz, Y2 Crystal

Commit message: PCB v0.2
Parts:
- added FID1, FID2, FID3: Fiducial, Fiducial:Fiducial_0.75mm_Mask2.25mm, symbol Mechanical:Fiducial
- added J10, J11, J12, J9: Conn_Coaxial, asl_footprints:GCT_RFPC-SMA27-F, symbol Connector:Conn_Coaxial
- added R2: 10 kΩ, Resistor_SMD:R_0603_1608Metric_Pad0.98x0.95mm_HandSolder, symbol Device:R_US
- added SW1: SW_DPDT_x2, asl_footprints:switch_slide_DPDT, symbol Switch:SW_DPDT_x2
- added U5: W25Q25PWSSIQ, Package_SON:WSON-8-1EP_8x6mm_P1.27mm_EP3.4x4.3mm, symbol Memory_Flash:W25Q128JVS
- C11, C12, C7, C8: value 10pF -> 10 pF
- C2, C3: value 10µF -> 10 µF; footprint Capacitor_SMD:C_1206_3216Metric -> Capacitor_SMD:C_1206_3216Metric_Pad1.33x1.80mm_HandSolder
- R1: value 20K -> 10 kΩ; footprint Resistor_SMD:R_1206_3216Metric -> Resistor_SMD:R_0603_1608Metric_Pad0.98x0.95mm_HandSolder
- renumbered D2 to D1, D1 to D2, H3 to H2, H2 to H3, J8 to J13, J9 to J14, J10 to J15, J11 to J16, J12 to J17, J13 to J18, J14 to J19, J15 to J20, J16 to J4, J4 to J5, J5 to J6, J6 to J7, J7 to J8, R2 to R3, R3 to R4, R6 to R5, R5 to R6, R4 to R7, U9 to U10, U10 to U11, U11 to U12, U12 to U13, U13 to U14, U14 to U15, U15 to U16, U16 to U17, U17 to U18, U18 to U19, U19 to U20, U20 to U21, U5 to U6, U6 to U7, U7 to U8, U8 to U9
Connections:
- net +12V: now also SW1.1 (A); no longer J2.1
- net +3.3V: now also U5.8 (VCC)
- net +5V: now also U2.3 (VI)
- net 11_A: now also U4.22 (PA0); no longer U4.34 (PB0)
- net 11_B: now also U4.23 (PA1)
- net 12_A: now also U4.83 (PD2)
- net 12_B: now also U4.81 (PD0)
- net 12_C: now also U4.82 (PD1)
- net 2_C: now also U4.77 (PA15); no longer U4.23 (PA1)
- net 2_COM_A: now also U4.34 (PB0); no longer U4.22 (PA0)
- net 3_C: now also J11.1 (In)
- net 8_C: now also J12.1 (In)
- net GND: now also J10.2 (Ext), J11.2 (Ext), J12.2 (Ext), J9.2 (Ext), SW1.3 (C), U5.4 (GND)
- net VBUS: no longer U2.3 (VI)
- net at RN1.11 (R6.2), U6.7 (~{HOLD}/~{RESET}/IO_{3}): now also U5.7 (~{HOLD}/~{RESET}/IO_{3})
- net at RN1.12 (R5.2), U6.3 (~{WP}/IO_{2}): now also U5.3 (~{WP}/IO_{2})
- net at RN1.13 (R4.2), U6.2 (DO/IO_{1}): now also U5.2 (DO/IO_{1})
- net at RN1.14 (R3.2), U6.5 (DI/IO_{0}): now also U5.5 (DI/IO_{0})
- net at RN1.15 (R2.2), U6.6 (CLK): now also U5.6 (CLK)
- net at RN1.16 (R1.2), U6.1 (~{CS}): now also U5.1 (~{CS})
- net at D2.2 (A): now also R2.2; no longer R1.2
- net SMA_1: now reaches U4.85 (PD4)
- net SMA_1: now also J9.1 (In)
- net SMA_2: now reaches U4.86 (PD5)
- net SMA_2: now also J10.1 (In)
- new net: R1.2, R2.1
- new net: J2.1, SW1.2 (B)
- no-connect marks 13 -> 7
Other:
- note added: "Indicator LEDs"
- moved on the sheet: C1, C2, C3, C4, C5, C6, D2, H1, H2, H3, H4, J2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

Commit message: PCB v0.3
don't short the power supply with the on/off switch 🤦
flipped UART4 pins. TX(4_A)/RX(4_B) was PC11(79)/PC10(78), now PC10(78)/PC11(79)
connect Vref to 3.3V so DAC works
change RGB LEDs to 10k
Parts:
- added C13: 100 nF, Capacitor_SMD:C_0603_1608Metric_Pad1.08x0.95mm_HandSolder, symbol Device:C_Small
- D1: value RGB_LED -> WP154A4SEJ3VBDZGW/CA
- D2: value 12_LED -> 151031VS06000
- H1, H2, H3, H4: value Threaded_Standoff -> 9774130360R
- J10, J11, J12, J9: value Conn_Coaxial -> RFPC-SMA27-F
- R1, R2, R3, R7: value 10 kΩ -> 10 KΩ
- R4, R5: value 91 Ω -> 10 KΩ
- R6: value 6.8Ω -> 10 KΩ
- S1, S2, S3: value TS02-66 -> TS02-66-170-BK-260-LCR-D
- SW1: value SW_DPDT_x2 -> 1825263-1
- U10, U11, U12, U13, U14, U15, U16, U17, U18, U19, U20, U21: value SRV05-4 -> D1213A-04TS-7
- U5: value W25Q25PWSSIQ -> W25Q256JVEIQ
Connections:
- net +12V: now also SW1.2 (B); no longer SW1.1 (A)
- net +3.3V: now also U4.20 (VREF+), C13.1
- net 4_A: now also U4.78 (PC10(UART4_TX)); no longer U4.79 (PC11(UART4_TX))
- net 4_B: now also U4.79 (PC11(UART4_RX)); no longer U4.78 (PC10(UART4_RX))
- net GND: now also C13.2; no longer SW1.3 (C)
- net at J2.1: now also SW1.3 (C); no longer SW1.2 (B)
- no-connect marks 7 -> 6
Other:
- moved on the sheet: C6, J3, R3, S1, S2, SW1A

Commit message: PCB v0.4
- was 2 layer, now 4 layer board
- was USB type B, now USB type C connector
- was SMA coaxial connectors, now BNC
- was 12 ports, now 10 ports
- added POW_C pins to 2 of the ports
- added8 extra GPIOs, 2 POW pins, and 5V/12V/GND rails on 16 pin terminal block
- 4 user buttons instead of 1
- 4 3mm LEDs instead of single RGB led
- removed SWD connector
- update to KiCAD 10
Parts:
- removed D1: WP154A4SEJ3VBDZGW/CA, LED_THT:LED_D5.0mm-4_RGB, symbol asl_symbols_new:RGB_LED
- removed J1: USB_B, asl_footprints:USB_B, symbol Connector:USB_B
- removed J3: SWD_connector, asl_footprints:SWD_2x5_socket, symbol asl_symbols_new:SWD_connector
- removed J4: Conn_01x06_Pin, Connector_PinHeader_2.54mm:PinHeader_1x06_P2.54mm_Vertical, symbol Connector:Conn_01x06_Pin
- removed J5, J6: RJ45_pyControl, asl_footprints:RJ45_THP_tab_on_top, symbol asl_symbols_new:RJ45_pyControl
- added D2, D3, D4, D5: 151031VS06000, LED_THT:LED_D3.0mm, symbol Device:LED
- added J2: USB4105-GF-A, Connector_USB:USB_C_Receptacle_GCT_USB4105-xx-A_16P_TopMnt_Horizontal, symbol asl_symbols_new:USB_C_Receptacle_USB2.0
- added J3: 1803413, Connector_Phoenix_MC:PhoenixContact_MC_1,5_16-G-3.81_1x16_P3.81mm_Horizontal, symbol Connector:Conn_01x16_Socket
- added R10, R12, R6, R9: 10 KΩ, Resistor_SMD:R_0603_1608Metric_Pad0.98x0.95mm_HandSolder, symbol Device:R_US
- added R2, R4: 5.1KΩ, Resistor_SMD:R_0603_1608Metric_Pad0.98x0.95mm_HandSolder, symbol Device:R_Small_US
- added S3, S4, S5: TS02-66-170-BK-260-LCR-D, asl_footprints:SW_TH_Tactile_TS02-66, symbol asl_symbols_new:TL3300
- DRA1, DRA2: value DIN_Rail_Adapter -> 1201578
- J10: renamed from J12; value RFPC-SMA27-F -> 0731000154; footprint asl_footprints:GCT_RFPC-SMA27-F -> asl_footprints:BNC RA Jack; Datasheet2 (none) -> https://www.digikey.com/short/hq32hv3d
- J11: renamed from J14; value RJ45_pyControl -> E5J88-00LJG2-L
- J12: renamed from J15; value RJ45_pyControl -> E5J88-00LJG2-L
- J13: renamed from J16; value RJ45_pyControl -> E5J88-00LJG2-L
- J14: renamed from J17; value RJ45_pyControl -> E5J88-00LJG2-L
- J15: renamed from J18; value RJ45_pyControl -> E5J88-00LJG2-L
- J16: renamed from J19; value RJ45_pyControl -> E5J88-00LJG2-L
- J17: renamed from J20; value RJ45_pyControl -> E5J88-00LJG2-L
- J4: renamed from J7; value RJ45_pyControl -> E5J88-00LJG2-L
- J5: renamed from J8; value RJ45_pyControl -> E5J88-00LJG2-L
- J6: renamed from J13; value RJ45_pyControl -> E5J88-00LJG2-L
- J7: renamed from J9; value RFPC-SMA27-F -> 0731000154; footprint asl_footprints:GCT_RFPC-SMA27-F -> asl_footprints:BNC RA Jack; Datasheet2 (none) -> https://www.digikey.com/short/hq32hv3d
- J8: renamed from J10; value RFPC-SMA27-F -> 0731000154; footprint asl_footprints:GCT_RFPC-SMA27-F -> asl_footprints:BNC RA Jack; Datasheet2 (none) -> https://www.digikey.com/short/hq32hv3d
- J9: renamed from J11; value RFPC-SMA27-F -> 0731000154; footprint asl_footprints:GCT_RFPC-SMA27-F -> asl_footprints:BNC RA Jack; Datasheet2 (none) -> https://www.digikey.com/short/hq32hv3d
- RN1: value 8x33Ω -> 8D33Ω
- Y2: value Crystal -> 32.768 KHz
- renumbered C9 to C10, C10 to C11, C11 to C12, C12 to C13, C13 to C8, C8 to C9, D2 to D1, J2 to J1, R6 to R11, R7 to R13, R2 to R3, R3 to R5, R4 to R7, R5 to R8, S3 to S6
Connections:
- net 11_C is gone; now on net 9_C: J16.5 (SPECIAL), U20.4 (IO3), U4.35 (PB1)
- net 11_COM_A is gone; now on net 9_COM_A: U4.54 (PB15), U9.3 (I3)
- net 11_COM_B is gone; now on net 9_COM_B: U4.55 (PD8), U9.4 (I4)
- net 11_PA is gone; now on net 9_PA: J16.3 (POW-A), U9.16 (O3)
- net 11_PB is gone; now on net 9_PB: J16.7 (POW-B), U9.15 (O4)
- net 12_C is gone; now on net 10_C: J17.5 (SPECIAL), U21.4 (IO3), U4.82 (PD1)
- net 12_COM_A is gone; now on net 10_COM_A: U4.40 (PE10), U9.1 (I1)
- net 12_COM_B is gone; now on net 10_COM_B: U4.45 (PE15), U9.2 (I2)
- net 12_PA is gone; now on net 10_PA: J17.3 (POW-A), U9.18 (O1)
- net 12_PB is gone; now on net 10_PB: J17.7 (POW-B), U9.17 (O2)
- net 3_C is gone; now on net 1_C: J4.5 (SPECIAL), J9.1 (In), U12.4 (IO3), U4.28 (PA4(DAC1,I2S1_WS))
- net +12V: now also J3.3 (Pin_3)
- net +3.3V: now also D2.2 (A), D3.2 (A), D4.2 (A), D5.2 (A), S3.3 (out1), S3.4 (out2), S4.3 (out1), S4.4 (out2), S5.3 (out1), S5.4 (out2)
- net +5V: now also J3.2 (Pin_2)
- net 10_A: now also J17.1 (DIO-A), U21.1 (IO1), U4.24 (PA2(UART2_TX)); no longer J15.1 (DIO-A), U19.1 (IO1), U4.44 (PE14(SPI4_MOSI))
- net 10_B: now also J17.4 (DIO-B), U21.3 (IO2), U4.25 (PA3(UART2_RX)); no longer J15.4 (DIO-B), U19.3 (IO2), U4.43 (PE13(SPI4_MISO))
- net 10_C: no longer J15.5 (SPECIAL), U19.4 (IO3), U4.42 (PE12(SPI4_SCK))
- net 10_COM_A: no longer U4.56 (PD9), U9.5 (I5)
- net 10_COM_B: no longer U4.57 (PD10), U9.6 (I6)
- net 10_PA: no longer J15.3 (POW-A), U9.14 (O5)
- net 10_PB: no longer J15.7 (POW-B), U9.13 (O6)
- net 1_A: now also J4.1 (DIO-A), U12.1 (IO1), U4.46 (PB10(UART3_TX,_I2C2_SCL)); no longer U10.1 (IO1), U4.68 (PA9(UART1_TX))
- net 1_B: now also J4.4 (DIO-B), U12.3 (IO2), U4.47 (PB11(UART3_RX,_I2C2_SDA)); no longer U10.3 (IO2), U4.69 (PA10(UART1_RX))
- net 1_C: no longer U10.4 (IO3), U4.67 (PA8)
- net 1_COM_A: now also U4.17 (PC2), U7.3 (I3); no longer U4.32 (PC4), U7.7 (I7)
- net 1_COM_B: now also U4.18 (PC3), U7.4 (I4); no longer U4.33 (PC5), U7.8 (I8)
- net 1_PA: now also J4.3 (POW-A), U7.16 (O3); no longer U7.12 (O7)
- net 1_PB: now also J4.7 (POW-B), U7.15 (O4); no longer U7.11 (O8)
- net 2_A: now also J5.1 (DIO-A), U13.1 (IO1), U4.78 (PC10(UART4_TX)); no longer U11.1 (IO1), U4.24 (PA2(UART2_TX))
- net 2_B: now also J5.4 (DIO-B), U13.3 (IO2), U4.79 (PC11(UART4_RX)); no longer U11.3 (IO2), U4.25 (PA3(UART2_RX))
- net 2_COM_A: now also U4.4 (PE5), U7.1 (I1); no longer U4.34 (PB0), U7.5 (I5)
- net 2_COM_B: now also U4.5 (PE6), U7.2 (I2); no longer U4.84 (PD3), U7.6 (I6)
- net 2_PA: now also J5.3 (POW-A), U7.18 (O1); no longer U7.14 (O5)
- net 2_PB: now also J5.7 (POW-B), U7.17 (O2); no longer U7.13 (O6)
- net 3_A: now also J6.1 (DIO-A), U14.1 (IO1), U4.52 (PB13(UART5_TX)); no longer J4.1 (DIO-A), U12.1 (IO1), U4.46 (PB10(UART3_TX,_I2C2_SCL))
- net 3_B: now also J6.4 (DIO-B), U14.3 (IO2), U4.51 (PB12(UART5_RX)); no longer J4.4 (DIO-B), U12.3 (IO2), U4.47 (PB11(UART3_RX,_I2C2_SDA))
- net 3_COM_A: now also U4.98 (PE1), U8.7 (I7); no longer U4.17 (PC2), U7.3 (I3)
- net 3_COM_B: now also U4.3 (PE4), U8.8 (I8); no longer U4.18 (PC3), U7.4 (I4)
- net 3_PA: now also J6.3 (POW-A), U8.12 (O7); no longer J4.3 (POW-A), U7.16 (O3)
- net 3_PB: now also J6.7 (POW-B), U8.11 (O8); no longer J4.7 (POW-B), U7.15 (O4)
- net 4_A: now also J11.1 (DIO-A), U15.1 (IO1), U4.63 (PC6(UART6_TX)); no longer J5.1 (DIO-A), U13.1 (IO1), U4.78 (PC10(UART4_TX))
- net 4_B: now also J11.4 (DIO-B), U15.3 (IO2), U4.64 (PC7(UART6_RX)); no longer J5.4 (DIO-B), U13.3 (IO2), U4.79 (PC11(UART4_RX))
- net 4_C: now also J11.5 (SPECIAL), U15.4 (IO3), U4.65 (PC8); no longer J5.5 (SPECIAL), U13.4 (IO3), U4.80 (PC12)
- net 4_COM_A: now also U4.15 (PC0), U8.5 (I5); no longer U4.4 (PE5), U7.1 (I1)
- net 4_COM_B: now also U4.97 (PE0), U8.6 (I6); no longer U4.5 (PE6), U7.2 (I2)
- net 4_PA: now also J11.3 (POW-A), U8.14 (O5); no longer J5.3 (POW-A), U7.18 (O1)
- net 4_PB: now also J11.7 (POW-B), U8.13 (O6); no longer J5.7 (POW-B), U7.17 (O2)
- net 5_A: now also J12.1 (DIO-A), U16.1 (IO1), U4.38 (PE8(UART7_TX)); no longer J6.1 (DIO-A), U14.1 (IO1), U4.52 (PB13(UART5_TX))
- net 5_B: now also J12.4 (DIO-B), U16.3 (IO2), U4.37 (PE7(UART7_RX)); no longer J6.4 (DIO-B), U14.3 (IO2), U4.51 (PB12(UART5_RX))
- net 5_C: now also J12.5 (SPECIAL), U16.4 (IO3), U4.39 (PE9); no longer J6.5 (SPECIAL), U14.4 (IO3), U4.53 (PB14)
- net 5_COM_A: now also U4.93 (PB7), U8.3 (I3); no longer U4.98 (PE1), U8.7 (I7)
- net 5_COM_B: now also U4.16 (PC1), U8.4 (I4); no longer U4.3 (PE4), U8.8 (I8)
- net 5_PA: now also J12.3 (POW-A), U8.16 (O3); no longer J6.3 (POW-A), U8.12 (O7)
- net 5_PB: now also J12.7 (POW-B), U8.15 (O4); no longer J6.7 (POW-B), U8.11 (O8)
- net 6_A: now also J13.1 (DIO-A), U17.1 (IO1), U4.95 (PB8(I2C1_SCL,CAN1_RX)); no longer J11.1 (DIO-A), U15.1 (IO1), U4.63 (PC6(UART6_TX))
- net 6_B: now also J13.4 (DIO-B), U17.3 (IO2), U4.96 (PB9(I2C1_SDA,CAN1_TX)); no longer J11.4 (DIO-B), U15.3 (IO2), U4.64 (PC7(UART6_RX))
- net 6_C: now also J10.1 (In), J13.5 (SPECIAL), U17.4 (IO3), U4.29 (PA5(DAC2,I2S1_CK)); no longer J11.5 (SPECIAL), U15.4 (IO3), U4.65 (PC8)
- net 6_COM_A: now also U4.87 (PD6), U8.1 (I1); no longer U4.15 (PC0), U8.5 (I5)
- net 6_COM_B: now also U4.88 (PD7), U8.2 (I2); no longer U4.97 (PE0), U8.6 (I6)
- net 6_PA: now also J13.3 (POW-A), U8.18 (O1); no longer J11.3 (POW-A), U8.14 (O5)
- net 6_PB: now also J13.7 (POW-B), U8.17 (O2); no longer J11.7 (POW-B), U8.13 (O6)
- net 7_A: now also J14.1 (DIO-A), U18.1 (IO1), U4.91 (PB5(SPI3_MOSI)); no longer J12.1 (DIO-A), U16.1 (IO1), U4.38 (PE8(UART7_TX))
- net 7_B: now also J14.4 (DIO-B), U18.3 (IO2), U4.90 (PB4(SPI3_MISO)); no longer J12.4 (DIO-B), U16.3 (IO2), U4.37 (PE7(UART7_RX))
- net 7_C: now also J14.5 (SPECIAL), U18.4 (IO3), U4.89 (PB3(SPI3_SCK)); no longer J12.5 (SPECIAL), U16.4 (IO3), U4.39 (PE9)
- net 7_COM_A: now also U4.61 (PD14), U9.7 (I7); no longer U4.93 (PB7), U8.3 (I3)
- net 7_COM_B: now also U4.62 (PD15), U9.8 (I8); no longer U4.16 (PC1), U8.4 (I4)
- net 7_PA: now also J14.3 (POW-A), U9.12 (O7); no longer J12.3 (POW-A), U8.16 (O3)
- net 7_PB: now also J14.7 (POW-B), U9.11 (O8); no longer J12.7 (POW-B), U8.15 (O4)
- net 8_A: now also J15.1 (DIO-A), U19.1 (IO1), U4.44 (PE14(SPI4_MOSI)); no longer J13.1 (DIO-A), U17.1 (IO1), U4.95 (PB8(I2C1_SCL,CAN1_RX))
- net 8_B: now also J15.4 (DIO-B), U19.3 (IO2), U4.43 (PE13(SPI4_MISO)); no longer J13.4 (DIO-B), U17.3 (IO2), U4.96 (PB9(I2C1_SDA,CAN1_TX))
- net 8_C: now also J15.5 (SPECIAL), U19.4 (IO3), U4.42 (PE12(SPI4_SCK)); no longer J10.1 (In), J13.5 (SPECIAL), U17.4 (IO3), U4.29 (PA5(DAC2,I2S1_CK))
- net 8_COM_A: now also U4.56 (PD9), U9.5 (I5); no longer U4.87 (PD6), U8.1 (I1)
- net 8_COM_B: now also U4.57 (PD10), U9.6 (I6); no longer U4.88 (PD7), U8.2 (I2)
- net 8_PA: now also J15.3 (POW-A), U9.14 (O5); no longer J13.3 (POW-A), U8.18 (O1)
- net 8_PB: now also J15.7 (POW-B), U9.13 (O6); no longer J13.7 (POW-B), U8.17 (O2)
- net 9_A: now also J16.1 (DIO-A), U20.1 (IO1), U4.68 (PA9(UART1_TX)); no longer J14.1 (DIO-A), U18.1 (IO1), U4.91 (PB5(SPI3_MOSI))
- net 9_B: now also J16.4 (DIO-B), U20.3 (IO2), U4.69 (PA10(UART1_RX)); no longer J14.4 (DIO-B), U18.3 (IO2), U4.90 (PB4(SPI3_MISO))
- net 9_C: no longer J14.5 (SPECIAL), U18.4 (IO3), U4.89 (PB3(SPI3_SCK))
- net 9_COM_A: no longer U4.61 (PD14), U9.7 (I7)
- net 9_COM_B: no longer U4.62 (PD15), U9.8 (I8)
- net 9_PA: no longer J14.3 (POW-A), U9.12 (O7)
- net 9_PB: no longer J14.7 (POW-B), U9.11 (O8)
- net GND: now also J2.A1 (GND), J2.A12 (GND), J2.B1 (GND), J2.B12 (GND), J2.S1 (SHIELD), J3.1 (Pin_1), J3.16 (Pin_16), J3.4 (Pin_4), J3.7 (Pin_7), R12.1, R2.2, R4.1, R6.1, R9.1
- net VBUS: now also J2.A4 (VBUS), J2.A9 (VBUS), J2.B4 (VBUS), J2.B9 (VBUS)
- net D8: now reaches U11.6 (IO4)
- net D8: now also U4.53 (PB14), J3.15 (Pin_15)
- net D3: now reaches U4.30 (PA6(I2S1_SDI))
- net D3: now also U10.4 (IO3), J3.10 (Pin_10)
- net D4: now reaches U4.31 (PA7(I2S1_SDO))
- net D4: now also U10.6 (IO4), J3.11 (Pin_11)
- net at U3.1 (I/O1): now also J2.B7 (D-)
- net at U3.3 (I/O2): now also J2.B6 (D+)
- removed net 11_A: J16.1 (DIO-A), U20.1 (IO1), U4.22 (PA0)
- removed net 11_B: J16.4 (DIO-B), U20.3 (IO2), U4.23 (PA1)
- removed net 12_A: J17.1 (DIO-A), U21.1 (IO1), U4.83 (PD2)
- removed net 12_B: J17.4 (DIO-B), U21.3 (IO2), U4.81 (PD0)
- net 2_C renamed D7
- net D7: now also J3.14 (Pin_14)
- net LED_1: no longer names the net of R7.1
- net LED_1: now also D2.1 (K)
- net LED_2: no longer names the net of R11.2
- net LED_2: now also D5.1 (K)
- net LED_3: no longer names the net of R8.1
- net LED_3: now also D3.1 (K)
- net SWCLK renamed D6
- net D6: now also U11.3 (IO2), J3.13 (Pin_13)
- net SWDIO renamed D5
- net D5: now also U11.1 (IO1), J3.12 (Pin_12)
- new net: R10.1, U4.83 (PD2)
- new net: D4.1 (K), R10.2
- new net: J2.A5 (CC1), R2.1
- new net: R6.2, S3.1 (in1), S3.2 (in2), U4.67 (PA8)
- new net: R12.2, S5.1 (in1), S5.2 (in2), U4.80 (PC12)
- new net: R9.2, S4.1 (in1), S4.2 (in2), U4.81 (PD0)
- new net: J2.B5 (CC2), R4.2
- new net 2_COM_C: U4.84 (PD3), U7.6 (I6)
- new net 2_PC: J5.5 (SPECIAL), U7.13 (O6)
- new net 3_COM_C: U4.34 (PB0), U7.5 (I5)
- new net 3_PC: J6.5 (SPECIAL), U7.14 (O5)
- new net D1: J3.8 (Pin_8), U10.1 (IO1), U4.22 (PA0)
- new net D2: J3.9 (Pin_9), U10.3 (IO2), U4.23 (PA1)
- new net P1: J3.5 (Pin_5), U7.12 (O7)
- new net P2: J3.6 (Pin_6), U7.11 (O8)
- new net X_COM_A: U4.32 (PC4), U7.7 (I7)
- new net X_COM_B: U4.33 (PC5), U7.8 (I8)
- no-connect marks 6 -> 21
Other:
- note added: "Auxiliary Header"
- note added: "BNC Connectors"
- note removed: "Indicator LEDs"
- moved on the sheet: C1, C12, C13, C6, C7, C9, J10, J7, J8, J9, R13, RN1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

Commit message: PCB v0.5
- connect USB-C shield ground
- connect A6/B6 and A7/B7 on USB-C
- connect C13 to ground
- use 5.1K resistors for everything
- make DC-DC converter pads smaller
- added QR code
- make GPIO labels larger and put on bottom side as well
- shift reset button to bottom right corner
- removed 2 of standoffs. shifted other two to be in vertical center of the board
- DIN connectors are now vertically centered
- added JST SH connector for I2C
- shifted terminal block up so it overhangs board (will stick out case)
- shifted dc jack and on off switch and dfu button and power LED
Parts:
- removed H3, H4: 9774130360R, asl_footprints:standoff_nut, symbol asl_symbols_new:Threaded_Standoff
- added J8: Conn_01x04_Socket, Connector_JST:JST_SH_SM04B-SRSS-TB_1x04-1MP_P1.00mm_Horizontal, symbol Connector:Conn_01x04_Socket
- added R10, R14, R15, R17, R4, R5: 5.1KΩ, Resistor_SMD:R_0603_1608Metric_Pad0.98x0.95mm_HandSolder, symbol Device:R_US
- R1: value 10 KΩ -> 5.1KΩ
- R11: renamed from R8; value 10 KΩ -> 5.1KΩ
- R12: renamed from R9; value 10 KΩ -> 5.1KΩ
- R13: renamed from R10; value 10 KΩ -> 5.1KΩ
- R16: renamed from R11; value 10 KΩ -> 5.1KΩ
- R18: renamed from R12; value 10 KΩ -> 5.1KΩ
- R19: renamed from R13; value 10 KΩ -> 5.1KΩ
- R2: renamed from R3; value 10 KΩ -> 5.1KΩ
- R7: renamed from R5; value 10 KΩ -> 5.1KΩ
- R8: renamed from R6; value 10 KΩ -> 5.1KΩ
- R9: renamed from R7; value 10 KΩ -> 5.1KΩ
- renumbered J7 to J1, J5 to J10, J6 to J11, J11 to J12, J12 to J13, J13 to J14, J14 to J15, J15 to J16, J16 to J17, J17 to J18, J8 to J2, J9 to J3, J10 to J4, J1 to J5, J2 to J6, J3 to J7, J4 to J9, R2 to R3, R4 to R6
Connections:
- net +3.3V: now also J8.2 (Pin_2)
- net 1_A: now also J8.4 (Pin_4)
- net 1_B: now also J8.3 (Pin_3)
- net GND: now also J6.SH (SHIELD), J8.1 (Pin_1); no longer J6.S1 (SHIELD)
- net at R13.1: now also R14.2; no longer U4.83 (PD2)
- net at R2.2: now also R5.1; no longer D1.2 (A)
- net at R9.2, U4.2 (PE3): now also R10.2
- net at R16.1, U4.66 (PC9): now also R17.1
- net at D2.1 (K), R9.1: now also R10.1
- net at D5.1 (K), R16.2: now also R17.2
- net SMA_1 renamed BNC_1
- net SMA_2 renamed BNC_2
- new net: R4.1, R5.2
- new net: D1.2 (A), R4.2
- new net: R15.1, U4.83 (PD2)
- new net: R14.1, R15.2
Other:
- note added: "Qwiic Stemma QT Modulino"
- note added: "SCL"
- note added: "SDA"
- moved on the sheet: D1, D2, D4, D5, J7, R1, R13, R16, R2, R8, R9, S3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

Commit message: PCB v0.6
Parts:
- removed R15, R2, R4, R5: 5.1KΩ, Resistor_SMD:R_0603_1608Metric_Pad0.98x0.95mm_HandSolder, symbol Device:R_US
- added R10, R12, R7: 5.1KΩ, Resistor_SMD:R_0603_1608Metric_Pad0.98x0.95mm_HandSolder, symbol Device:R_US
- D3: value 151031VS06000 -> 151031SS06000
- D4: value 151031VS06000 -> 151033BS03000
- D5: value 151031VS06000 -> 151031YS05900
- R1, R13: value 5.1KΩ -> 20K
- renumbered R12 to R11, R16 to R15, R17 to R16, R18 to R17, R19 to R18, R3 to R2, R6 to R3, R7 to R4, R8 to R5, R9 to R6, R10 to R8, R11 to R9
Connections:
- net at R13.1: now also R12.2; no longer R14.2
- net at R13.2: now also U4.83 (PD2); no longer D4.1 (K)
- net at D3.1 (K), R9.1: now also R10.1
- net at D1.2 (A): now also R1.2
- net at R14.1: now also R15.1, R16.1, U4.66 (PC9)
- net at R6.2, R8.2, U4.2 (PE3): now also R7.2
- net at R9.2, U4.41 (PE11): now also R10.2
- net at J6.B7 (D-), U3.1 (I/O1): now also J6.A7 (D-)
- net at J6.B6 (D+), U3.3 (I/O2): now also J6.A6 (D+)
- net at D2.1 (K), R6.1, R8.1: now also R7.1
- net at D5.1 (K), R15.2, R16.2: now also R14.2
- new net: D4.1 (K), R12.1
- no-connect marks 21 -> 19
Other:
- note added: "Blue"
- note added: "Green"
- note added: "Red"
- note added: "Yellow"
- moved on the sheet: D1, D2, D3, D4, D5, R1, R16, R8, R9
