File: pcb/h7_breakout.kicad_sch (KiCad schematic)
At the start: 92 parts, among them J1 0731000154, J10 E5J88-00LJG2-L, J11 E5J88-00LJG2-L, J12 E5J88-00LJG2-L, J13 E5J88-00LJG2-L, J14 E5J88-00LJG2-L, J15 E5J88-00LJG2-L, J16 E5J88-00LJG2-L, J17 E5J88-00LJG2-L, J18 E5J88-00LJG2-L, J2 0731000154, J3 0731000154, J4 0731000154, J5 PJ-037A, J6 USB4105-GF-A, J7 1803413, J8 Conn_01x04_Socket, J9 E5J88-00LJG2-L, SW1 1825263-1, U1 R-78E5.0-1.0, U10 D1213A-04TS-7, U11 D1213A-04TS-7, U12 D1213A-04TS-7, U13 D1213A-04TS-7, U14 D1213A-04TS-7, U15 D1213A-04TS-7, U16 D1213A-04TS-7, U17 D1213A-04TS-7, U18 D1213A-04TS-7, U19 D1213A-04TS-7, U2 AMS1117-3.3, U20 D1213A-04TS-7, U21 D1213A-04TS-7, U3 USBLC6-2SC6, U4 STM32H743VIT6, U5 W25Q256JVEIQ, U6 W25Q25PWSSIQ, U7 TBD62083APG, U8 TBD62083APG, U9 TBD62083APG, Y1 25 MHz, Y2 32.768 KHz

Commit message: PCB v0.7
Parts:
- added TP1: 5019, TestPoint:TestPoint_Keystone_5019_Miniature, symbol Connector:TestPoint
- added U12: D1213A-04TS-7, Package_TO_SOT_SMD:SOT-23-6, symbol Power_Protection:SRV05-4
- D1: value 151031VS06000 -> 151031SS06000
- J7: renamed from J8; value Conn_01x04_Socket -> SM04B-SRSS-TB
- R1, R13: value 20K -> 20 KΩ
- R10, R11, R12, R14, R15, R16, R17, R18, R2, R3, R4, R5, R6, R7, R8, R9: value 5.1KΩ -> 5.1 KΩ
- RN1: value 8D33Ω -> 33 Ω
- S1, S2, S3, S4, S5, S6: footprint asl_footprints:SW_TH_Tactile_TS02-66 -> asl_footprints:SW_TH_Tactile_TS02-66-170
- Y2: value 32.768 KHz -> 32.768 kHz
- renumbered C13 to C12, C12 to C13, J5 to J1, J1 to J2, J2 to J3, J3 to J4, J4 to J5, J7 to J8, U12 to U13, U13 to U14, U14 to U15, U15 to U16, U16 to U17, U17 to U18, U18 to U19, U19 to U20, U20 to U21, U21 to U22
Connections:
- net +3.3V: now also U12.5 (VP)
- net BNC_1: now also U12.6 (IO4)
- net BNC_2: now also U12.4 (IO3)
- net GND: now also TP1.1, U12.2 (VN)
Other:
- note added: "BNT_A"
- note added: "BNT_D"
- note added: "BTN_B"
- note added: "BTN_C"
- note added: "Plug link"
- note removed: "USER"
- company: (none) -> Andy Lustig
- moved on the sheet: C10, C12, C13, C2, C3, C4, C5, C6, D1, D2, D3, D5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

Commit message: pcb v0.8
Parts:
- removed C2, C3: 10 µF, Capacitor_SMD:C_1206_3216Metric_Pad1.33x1.80mm_HandSolder, symbol Device:C
- removed C4: 10 µF, Capacitor_SMD:C_1206_3216Metric_Pad1.33x1.80mm_HandSolder, symbol Device:C_Small
- removed C5: 100 nF, Capacitor_SMD:C_0603_1608Metric_Pad1.08x0.95mm_HandSolder, symbol Device:C_Small
- removed J2, J3: 0731000154, asl_footprints:BNC RA Jack, symbol Connector:Conn_Coaxial
- removed J8: 1803413, Connector_Phoenix_MC:PhoenixContact_MC_1,5_16-G-3.81_1x16_P3.81mm_Horizontal, symbol Connector:Conn_01x16_Socket
- removed R5: 5.1 KΩ, Resistor_SMD:R_0603_1608Metric_Pad0.98x0.95mm_HandSolder, symbol Device:R_US
- removed RN1: 33 Ω, Package_SO:SSOP-16_3.9x4.9mm_P0.635mm, symbol Device:R_Pack08
- removed S3, S4: TS02-66-170-BK-260-LCR-D, asl_footprints:SW_TH_Tactile_TS02-66-170, symbol asl_symbols_new:TL3300
- removed U11, U12: D1213A-04TS-7, Package_TO_SOT_SMD:SOT-23-6, symbol Power_Protection:SRV05-4
- added C2: 10 µF, Capacitor_SMD:C_1206_3216Metric_Pad1.33x1.80mm_HandSolder, symbol Device:C_Small
- added C3: 100 nF, Capacitor_SMD:C_0603_1608Metric_Pad1.08x0.95mm_HandSolder, symbol Device:C_Small
- added C4, C5: 10 µF, Capacitor_SMD:C_1206_3216Metric_Pad1.33x1.80mm_HandSolder, symbol Device:C
- added D2: 151031SS06000, LED_THT:LED_D3.0mm, symbol Device:LED
- added H3, H4: 7790, asl_footprints:RA_screw_mount, symbol asl_symbols_new:Threaded_Standoff
- added J6: 1803332, Connector_Phoenix_MC:PhoenixContact_MC_1,5_8-G-3.81_1x08_P3.81mm_Horizontal, symbol Connector:Conn_01x08_Socket
- added JP1, JP2, JP3, JP4: M20-9990246, Connector_PinHeader_2.54mm:PinHeader_1x02_P2.54mm_Vertical, symbol Jumper:Jumper_2_Open
- added R12, R13, R14, R15, R16, R20, R22, R23, R25, R27, R28, R29, R30, R31, R32, R33, R34, R35, R36, R39, R40, R41, R42, R43, R46, R47, R50, R52, R6, R7, R8, R9: 100 Ω, Resistor_SMD:R_0603_1608Metric_Pad0.98x0.95mm_HandSolder, symbol Device:R_US
- added R2, R21, R44: 5.1 KΩ, Resistor_SMD:R_0603_1608Metric_Pad0.98x0.95mm_HandSolder, symbol Device:R_US
- added R3: 20 KΩ, Resistor_SMD:R_0603_1608Metric_Pad0.98x0.95mm_HandSolder, symbol Device:R_US
- added R51, R53, R54, R55, R57, R58: 33 Ω, Resistor_SMD:R_0603_1608Metric_Pad0.98x0.95mm_HandSolder, symbol Device:R_US
- added SW2, SW3: PTS645VL58-2 LFS, Button_Switch_THT:SW_Tactile_SPST_Angled_PTS645Vx58-2LFS, symbol Switch:SW_MEC_5G
- J1: value PJ-037A -> PJ-037AH
- R1: value 20 KΩ -> 5.1 KΩ
- R11: value 5.1 KΩ -> 100 Ω
- SW1: footprint asl_footprints:switch_slide_DPDT -> asl_footprints:RA toggle
- U1: value R-78E5.0-1.0 -> TSR 3-2450N; footprint asl_footprints:Converter_DCDC_RECOM_R-78E-0.5_THT -> asl_footprints:Converter_DCDC_traco_3A
- U10: LCSC (none) -> C460588
- U11: renamed from U13; LCSC (none) -> C460588
- U12: renamed from U14; LCSC (none) -> C460588
- U13: renamed from U15; LCSC (none) -> C460588
- U14: renamed from U16; LCSC (none) -> C460588
- U15: renamed from U17; LCSC (none) -> C460588
- U16: renamed from U18; LCSC (none) -> C460588
- U17: renamed from U19; LCSC (none) -> C460588
- U18: renamed from U20; LCSC (none) -> C460588
- U19: renamed from U21; LCSC (none) -> C460588
- U20: renamed from U22; LCSC (none) -> C460588
- U3: LCSC (none) -> C7519
- U4: LCSC (none) -> C114409
- U5: LCSC (none) -> C97522
- U7, U8, U9: value TBD62083APG -> TBD62083AFNG,EL; LCSC (none) -> C163229
- renumbered D2 to D3, D3 to D4, D4 to D5, D5 to D6, J12 to J10, J13 to J11, J14 to J12, J15 to J13, J16 to J14, J17 to J15, J18 to J16, J4 to J2, J5 to J3, J6 to J4, J7 to J5, J9 to J7, J10 to J8, J11 to J9, R4 to R10, R6 to R17, R7 to R18, R8 to R19, R9 to R24, R10 to R26, R12 to R37, R13 to R38, R2 to R4, R14 to R45, R15 to R48, R16 to R49, R3 to R5, R17 to R56, R18 to R59, S5 to S3, S6 to S4
Connections:
- net +12V: now also C4.1, J6.3 (Pin_3), R3.1; no longer R1.1
- net +3.3V: now also R1.1, S2.3 (out1), S2.4 (out2), C2.1, C3.1, R2.1, SW2.2 (A), SW2.4 (B)
- net +5V: now also C5.1, J6.2 (Pin_2); no longer U2.3 (VI)
- net 10_A: now also R8.2; no longer U4.24 (PA2(UART2_TX))
- net 10_B: now also R9.2; no longer U4.25 (PA3(UART2_RX))
- net 10_C: now also R35.1; no longer U4.82 (PD1)
- net 1_A: now also R36.2; no longer U4.46 (PB10(UART3_TX,_I2C2_SCL))
- net 1_B: now also R39.2; no longer U4.47 (PB11(UART3_RX,_I2C2_SDA))
- net 1_C: now also R11.2, JP3.1 (A); no longer J2.1 (In), U4.28 (PA4(DAC1,I2S1_WS))
- net 2_A: now also R6.2; no longer U4.78 (PC10(UART4_TX))
- net 2_B: now also R7.2; no longer U4.79 (PC11(UART4_RX))
- net 3_A: now also R41.2; no longer U4.52 (PB13(UART5_TX))
- net 3_B: now also R40.2; no longer U4.51 (PB12(UART5_RX))
- net 4_A: now also R46.2; no longer U4.63 (PC6(UART6_TX))
- net 4_B: now also R47.2; no longer U4.64 (PC7(UART6_RX))
- net 4_C: now also R43.2; no longer U4.65 (PC8)
- net 5_A: now also R22.1; no longer U4.38 (PE8(UART7_TX))
- net 5_B: now also R20.1; no longer U4.37 (PE7(UART7_RX))
- net 5_C: now also R23.1; no longer U4.39 (PE9)
- net 6_A: now also R32.2; no longer U4.95 (PB8(I2C1_SCL,CAN1_RX))
- net 6_B: now also R34.2; no longer U4.96 (PB9(I2C1_SDA,CAN1_TX))
- net 6_C: now also JP4.1 (A), R12.2; no longer J3.1 (In), U4.29 (PA5(DAC2,I2S1_CK))
- net 7_A: now also R30.2; no longer U4.91 (PB5(SPI3_MOSI))
- net 7_B: now also R28.2; no longer U4.90 (PB4(SPI3_MISO))
- net 7_C: now also R25.2; no longer U4.89 (PB3(SPI3_SCK))
- net 8_A: now also R31.1; no longer U4.44 (PE14(SPI4_MOSI))
- net 8_B: now also R29.1; no longer U4.43 (PE13(SPI4_MISO))
- net 8_C: now also R27.1; no longer U4.42 (PE12(SPI4_SCK))
- net 9_A: now also R15.2; no longer U4.68 (PA9(UART1_TX))
- net 9_B: now also R16.2; no longer U4.69 (PA10(UART1_RX))
- net 9_C: now also R13.2; no longer U4.35 (PB1)
- net BNC_1: now also J2.1 (In), JP1.2 (B), JP3.2 (B); no longer U4.85 (PD4)
- net BNC_2: now also J3.1 (In), JP2.2 (B), JP4.2 (B); no longer U4.86 (PD5)
- net BOOT: now also SW2.1 (A), SW2.2 (A); no longer S1.1 (in1), S1.2 (in2)
- net D1: now also U10.3 (IO2), J6.6 (Pin_6), R50.2; no longer U10.1 (IO1), U4.22 (PA0)
- net D2: now also U10.1 (IO1), J6.7 (Pin_7), R52.2; no longer U10.3 (IO2), U4.23 (PA1)
- net D3: now also J6.8 (Pin_8), R14.2; no longer U4.30 (PA6(I2S1_SDI))
- net D4: now also JP1.1 (A), R33.1; no longer U10.6 (IO4), U4.31 (PA7(I2S1_SDO))
- net D5: now also JP2.1 (A), R42.1; no longer U4.72 (PA13)
- net GND: now also C2.2, C3.2, C4.2, C5.2, D2.1 (K), J6.1 (Pin_1), R21.1, R44.1, SW3.1 (A), SW3.2 (A); no longer R11.1, S2.1 (in1), S2.2 (in2)
- net P1: now also J6.4 (Pin_4)
- net P2: now also J6.5 (Pin_5)
- net Q_CLK: now also R53.2
- net Q_CS: now also R51.2
- net Q_DI: now also R54.2
- net Q_DO: now also R55.2
- net Q_HOLD: now also R58.2
- net Q_WP: now also R57.2
- net RST: now also SW3.2 (A), SW3.4 (B); no longer S2.3 (out1), S2.4 (out2)
- net VBUS: now also U2.3 (VI)
- net BTN_B: now reaches R56.2, S3.1 (in1), S3.2 (in2), U4.80 (PC12)
- net at U4.81 (PD0): now also R33.2; no longer R11.2
- net at U5.7 (~{HOLD}/~{RESET}/IO_{3}), U6.7 (~{HOLD}/~{RESET}/IO_{3}): now also R58.1
- net at U5.3 (~{WP}/IO_{2}), U6.3 (~{WP}/IO_{2}): now also R57.1
- net at U5.2 (DO/IO_{1}), U6.2 (DO/IO_{1}): now also R55.1
- net at U5.5 (DI/IO_{0}), U6.5 (DI/IO_{0}): now also R54.1
- net at U5.6 (CLK), U6.6 (CLK): now also R53.1
- net at U5.1 (~{CS}), U6.1 (~{CS}): now also R51.1
- net at D1.2 (A): now also R3.2; no longer R1.2
- net D6: no longer names the net of U4.76 (PA14)
- net D7 renamed BTN_D
- net BTN_D: now also S1.1 (in1), S1.2 (in2), R21.2
- net D8: no longer names the net of U4.53 (PB14)
- net D8: now also R43.1
- new net: R52.1, U4.79 (PC11(UART4_RX))
- new net: R28.1, U4.90 (PB4(SPI3_MISO))
- new net: R34.1, U4.96 (PB9(I2C1_SDA,CAN1_TX))
- new net: R30.1, U4.91 (PB5(SPI3_MOSI))
- new net: R42.2, U4.86 (PD5)
- new net: R36.1, U4.46 (PB10(UART3_TX,_I2C2_SCL))
- new net: D2.2 (A), R1.2, R2.2
- new net: R8.1, U4.24 (PA2(UART2_TX))
- new net: R32.1, U4.95 (PB8(I2C1_SCL,CAN1_RX))
- new net: R41.1, U4.52 (PB13(UART5_TX))
- new net: R40.1, U4.51 (PB12(UART5_RX))
- new net: R22.2, U4.38 (PE8(UART7_TX))
- new net: R13.1, U4.30 (PA6(I2S1_SDI))
- new net: R31.2, U4.44 (PE14(SPI4_MOSI))
- new net: R6.1, U4.22 (PA0)
- new net: R7.1, U4.23 (PA1)
- new net: R9.1, U4.25 (PA3(UART2_RX))
- new net: R11.1, U4.28 (PA4(DAC1,I2S1_WS))
- new net: R12.1, U4.29 (PA5(DAC2,I2S1_CK))
- new net: R14.1, U4.31 (PA7(I2S1_SDO))
- new net: R20.2, U4.37 (PE7(UART7_RX))
- new net: R23.2, U4.39 (PE9)
- new net: R27.2, U4.42 (PE12(SPI4_SCK))
- new net: R29.2, U4.43 (PE13(SPI4_MISO))
- new net: R39.1, U4.47 (PB11(UART3_RX,_I2C2_SDA))
- new net: R46.1, U4.63 (PC6(UART6_TX))
- new net: R47.1, U4.64 (PC7(UART6_RX))
- new net: R15.1, U4.68 (PA9(UART1_TX))
- new net: R16.1, U4.69 (PA10(UART1_RX))
- new net: R50.1, U4.78 (PC10(UART4_TX))
- new net: R35.2, U4.82 (PD1)
- new net: R25.1, U4.89 (PB3(SPI3_SCK))
- new net BTN_C: R44.2, S2.1 (in1), S2.2 (in2), U4.85 (PD4)
- no-connect marks 19 -> 20
Other:
- note added: "1"
- note added: "10"
- note added: "2"
- note added: "3"
- note added: "4"
- note added: "5"
- note added: "6"
- note added: "7"
- note added: "8"
- note added: "9"
- note added: "ENCODER"
- note added: "MCU"
- note added: "Power Drivers"
- note added: "jumper link"
- note removed: "Power Driver"
- moved on the sheet: D3, D4, D5, D6, DRA1, DRA2, FID1, FID2, FID3, H1, H2, J2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

Commit message: pcb v0.9
Parts:
- removed JP1, JP2, JP3, JP4: M20-9990246, Connector_PinHeader_2.54mm:PinHeader_1x02_P2.54mm_Vertical, symbol Jumper:Jumper_2_Open
- removed R32, R34, R36, R39: 100 Ω, Resistor_SMD:R_0603_1608Metric_Pad0.98x0.95mm_HandSolder, symbol Device:R_US
- added S5: CAS-D20TB, asl_footprints:CAS-D20TB, symbol asl_symbols_new:CAS-D20TB
- R11, R12, R13, R14, R15, R16, R20, R22, R23, R25, R27, R28, R29, R30, R31, R6, R7, R8, R9: value 100 Ω -> 33 Ω
- R32: renamed from R33; value 100 Ω -> 33 Ω
- R33: renamed from R35; value 100 Ω -> 33 Ω
- R36: renamed from R40; value 100 Ω -> 33 Ω
- R37: renamed from R41; value 100 Ω -> 33 Ω
- R38: renamed from R42; value 100 Ω -> 33 Ω
- R39: renamed from R43; value 100 Ω -> 33 Ω
- R42: renamed from R46; value 100 Ω -> 33 Ω
- R43: renamed from R47; value 100 Ω -> 33 Ω
- R46: renamed from R50; value 100 Ω -> 33 Ω
- R48: renamed from R52; value 100 Ω -> 33 Ω
- SW1: value 1825263-1 -> 100SP1T2B4M6QE
- TP1: footprint TestPoint:TestPoint_Keystone_5019_Miniature -> TestPoint:TestPoint_Plated_Hole_D2.0mm
- renumbered H3 to H2, H2 to H3, R37 to R34, R38 to R35, R44 to R40, R45 to R41, R48 to R44, R49 to R45, R51 to R47, R53 to R49, R54 to R50, R55 to R51, R56 to R52, R57 to R53, R58 to R54, R59 to R55
Connections:
- net +12V: now also J6.1 (Pin_1); no longer J6.3 (Pin_3)
- net +5V: now also J6.3 (Pin_3); no longer J6.2 (Pin_2)
- net 1_A: now also U4.46 (PB10(UART3_TX,_I2C2_SCL))
- net 1_B: now also U4.47 (PB11(UART3_RX,_I2C2_SDA))
- net 1_C: now also U11.6 (IO4), S5.1; no longer U11.4 (IO3)
- net 6_A: now also U4.95 (PB8(I2C1_SCL,CAN1_RX))
- net 6_B: now also U4.96 (PB9(I2C1_SDA,CAN1_TX))
- net 6_C: now also S5.4
- net BNC_1: now also S5.2
- net BNC_2: now also S5.5
- net D4: now also U10.6 (IO4), S5.3
- net D5: now also U11.4 (IO3), S5.6
- net GND: now also J6.7 (Pin_7); no longer J6.1 (Pin_1)
- net D1 renamed 11_A
- net 11_A: now also J6.8 (Pin_8); no longer J6.6 (Pin_6)
- net D2 renamed 11_B
- net 11_B: now also J6.5 (Pin_5); no longer J6.7 (Pin_7)
- net D3 renamed 11_C
- net 11_C: now also J6.4 (Pin_4); no longer J6.8 (Pin_8)
- net P1 renamed 11_PA
- net 11_PA: now also J6.6 (Pin_6); no longer J6.4 (Pin_4)
- net P2 renamed 11_PB
- net 11_PB: now also J6.2 (Pin_2); no longer J6.5 (Pin_5)
- net X_COM_A renamed 11_COM_A
- net X_COM_B renamed 11_COM_B
- no-connect marks 20 -> 19
Other:
- note added: "Auxiliary Header Port 11"
- note added: "DIN clips"
- note added: "Front standoffs"
- note added: "Top standoffs"
- note removed: "Auxiliary Header"
- note removed: "jumper link"
- moved on the sheet: DRA1, DRA2, FID1, FID2, FID3, H1, H2, H3, H4, J3, J5, J6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
