File: pcb/h7_breakout.kicad_pcb (KiCad board)
At the start: 4 copper layers, 253 x 52 mm, 92 parts, among them J1 0731000154, J10 E5J88-00LJG2-L, J11 E5J88-00LJG2-L, J12 E5J88-00LJG2-L, J13 E5J88-00LJG2-L, J14 E5J88-00LJG2-L, J15 E5J88-00LJG2-L, J16 E5J88-00LJG2-L, J17 E5J88-00LJG2-L, J18 E5J88-00LJG2-L, J2 0731000154, J3 0731000154, J4 0731000154, J5 PJ-037A, J6 USB4105-GF-A, J7 1803413, J8 Conn_01x04_Socket, J9 E5J88-00LJG2-L, SW1 1825263-1, U1 R-78E5.0-1.0, U10 D1213A-04TS-7, U11 D1213A-04TS-7, U12 D1213A-04TS-7, U13 D1213A-04TS-7, U14 D1213A-04TS-7, U15 D1213A-04TS-7, U16 D1213A-04TS-7, U17 D1213A-04TS-7, U18 D1213A-04TS-7, U19 D1213A-04TS-7, U2 AMS1117-3.3, U20 D1213A-04TS-7, U21 D1213A-04TS-7, U3 USBLC6-2SC6, U4 STM32H743VIT6, U5 W25Q256JVEIQ, U6 W25Q25PWSSIQ, U7 TBD62083APG, U8 TBD62083APG, U9 TBD62083APG, Y1 25 MHz, Y2 32.768 KHz

Commit message: PCB v0.7
Parts:
- added TP1: 5019, TestPoint:TestPoint_Keystone_5019_Miniature, F.Cu at (250.7, 102.7)
- added U12: D1213A-04TS-7, Package_TO_SOT_SMD:SOT-23-6, F.Cu at (46.7, 120.9)
- D1: value 151031VS06000 -> 151031SS06000
- J7: renamed from J8; value Conn_01x04_Socket -> SM04B-SRSS-TB
- R1, R13: value 20K -> 20 KΩ
- R10, R11, R12, R14, R15, R16, R17, R18, R2, R3, R4, R5, R6, R7, R8, R9: value 5.1KΩ -> 5.1 KΩ
- RN1: value 8D33Ω -> 33 Ω
- S1, S2, S3, S4, S5, S6: footprint asl_footprints:SW_TH_Tactile_TS02-66 -> asl_footprints:SW_TH_Tactile_TS02-66-170
- Y2: value 32.768 KHz -> 32.768 kHz
- moved S3 7.91 mm to (34.2, 117.6), turned to 180 degrees
- moved S1 3.95 mm to (233.3, 91.9)
- renumbered C13 to C12, C12 to C13, J5 to J1, J1 to J2, J2 to J3, J3 to J4, J4 to J5, J7 to J8, U12 to U13, U13 to U14, U14 to U15, U15 to U16, U16 to U17, U17 to U18, U18 to U19, U19 to U20, U20 to U21, U21 to U22
Routing:
- net /BNC_2: track 145.3 -> 152.9 mm
- net /BNC_1: track 174.3 -> 181.7 mm
- net GND: track 81.8 -> 87.5 mm, vias 43 -> 42
- net +3.3V: track 47.0 -> 51.9 mm
- net Net-(S3-in1): track 176.5 -> 172.0 mm
Other:
- board text added: "D10"
- board text added: "D9"
- board text added: "GND"
- board text added: "OFF"
- board text added: "ON"
- board text added: "v${REVISION} July 2026 AL"
- board text removed: "12"
- board text removed: "v${REVISION} June 2026"

Commit message: pcb v0.8
Parts:
- removed the C4 at (244.8, 112.7)
- removed the J2 at (38.8, 126.5)
- removed the J3 at (54.8, 126.5)
- removed the J8 at (101.8, 84.4)
- removed RN1: 33 Ω, Package_SO:SSOP-16_3.9x4.9mm_P0.635mm
- removed the S1 at (233.3, 91.9)
- removed the S2 at (268.2, 127.0)
- removed the U11 at (54.0, 96.8)
- removed the U12 at (46.7, 120.9)
- added C2: 10 µF, Capacitor_SMD:C_1206_3216Metric_Pad1.33x1.80mm_HandSolder, F.Cu at (237.2, 106.5)
- added D2: 151031SS06000, LED_THT:LED_D3.0mm, F.Cu at (233.0, 88.2)
- added H3: 7790, asl_footprints:RA_screw_mount, F.Cu at (61.0, 123.2)
- added H4: 7790, asl_footprints:RA_screw_mount, F.Cu at (264.7, 123.2)
- added J6: 1803332, Connector_Phoenix_MC:PhoenixContact_MC_1,5_8-G-3.81_1x08_P3.81mm_Horizontal, F.Cu at (102.1, 76.4)
- added JP1: M20-9990246, Connector_PinHeader_2.54mm:PinHeader_1x02_P2.54mm_Vertical, F.Cu at (80.5, 117.7)
- added JP2: M20-9990246, Connector_PinHeader_2.54mm:PinHeader_1x02_P2.54mm_Vertical, F.Cu at (96.5, 117.7)
- added JP3: M20-9990246, Connector_PinHeader_2.54mm:PinHeader_1x02_P2.54mm_Vertical, F.Cu at (80.5, 127.5)
- added JP4: M20-9990246, Connector_PinHeader_2.54mm:PinHeader_1x02_P2.54mm_Vertical, F.Cu at (96.5, 127.5)
- added R11: 100 Ω, Resistor_SMD:R_0603_1608Metric_Pad0.98x0.95mm_HandSolder, F.Cu at (119.9, 107.5)
- added R12: 100 Ω, Resistor_SMD:R_0603_1608Metric_Pad0.98x0.95mm_HandSolder, F.Cu at (159.0, 108.8)
- added R13: 100 Ω, Resistor_SMD:R_0603_1608Metric_Pad0.98x0.95mm_HandSolder, F.Cu at (231.5, 116.5)
- added R14: 100 Ω, Resistor_SMD:R_0603_1608Metric_Pad0.98x0.95mm_HandSolder, F.Cu at (97.5, 89.2)
- added R15: 100 Ω, Resistor_SMD:R_0603_1608Metric_Pad0.98x0.95mm_HandSolder, F.Cu at (227.5, 115.5)
- added R16: 100 Ω, Resistor_SMD:R_0603_1608Metric_Pad0.98x0.95mm_HandSolder, F.Cu at (228.8, 103.8)
- added R2: 5.1 KΩ, Resistor_SMD:R_0603_1608Metric_Pad0.98x0.95mm_HandSolder, F.Cu at (233.0, 94.0)
- added R20: 100 Ω, Resistor_SMD:R_0603_1608Metric_Pad0.98x0.95mm_HandSolder, F.Cu at (166.5, 116.5)
- added R22: 100 Ω, Resistor_SMD:R_0603_1608Metric_Pad0.98x0.95mm_HandSolder, F.Cu at (174.0, 116.0)
- added R23: 100 Ω, Resistor_SMD:R_0603_1608Metric_Pad0.98x0.95mm_HandSolder, F.Cu at (168.0, 113.5)
- added R25: 100 Ω, Resistor_SMD:R_0603_1608Metric_Pad0.98x0.95mm_HandSolder, F.Cu at (189.0, 86.8)
- added R27: 100 Ω, Resistor_SMD:R_0603_1608Metric_Pad0.98x0.95mm_HandSolder, F.Cu at (193.8, 110.2)
- added R28: 100 Ω, Resistor_SMD:R_0603_1608Metric_Pad0.98x0.95mm_HandSolder, F.Cu at (185.0, 85.5)
- added R29: 100 Ω, Resistor_SMD:R_0603_1608Metric_Pad0.98x0.95mm_HandSolder, F.Cu at (193.5, 113.8)
- added R3: 20 KΩ, Resistor_SMD:R_0603_1608Metric_Pad0.98x0.95mm_HandSolder, F.Cu at (243.8, 92.5)
- added R30: 100 Ω, Resistor_SMD:R_0603_1608Metric_Pad0.98x0.95mm_HandSolder, F.Cu at (175.2, 83.2)
- added R31: 100 Ω, Resistor_SMD:R_0603_1608Metric_Pad0.98x0.95mm_HandSolder, F.Cu at (189.5, 111.2)
- added R32: 100 Ω, Resistor_SMD:R_0603_1608Metric_Pad0.98x0.95mm_HandSolder, F.Cu at (177.8, 81.2)
- added R33: 100 Ω, Resistor_SMD:R_0603_1608Metric_Pad0.98x0.95mm_HandSolder, F.Cu at (158.2, 78.8)
- added R34: 100 Ω, Resistor_SMD:R_0603_1608Metric_Pad0.98x0.95mm_HandSolder, F.Cu at (173.8, 79.8)
- added R35: 100 Ω, Resistor_SMD:R_0603_1608Metric_Pad0.98x0.95mm_HandSolder, F.Cu at (241.8, 116.2)
- added R36: 100 Ω, Resistor_SMD:R_0603_1608Metric_Pad0.98x0.95mm_HandSolder, F.Cu at (114.0, 111.5)
- added R39: 100 Ω, Resistor_SMD:R_0603_1608Metric_Pad0.98x0.95mm_HandSolder, F.Cu at (119.1, 112.5)
- added R40: 100 Ω, Resistor_SMD:R_0603_1608Metric_Pad0.98x0.95mm_HandSolder, F.Cu at (141.7, 113.8)
- added R41: 100 Ω, Resistor_SMD:R_0603_1608Metric_Pad0.98x0.95mm_HandSolder, F.Cu at (147.1, 113.3)
- added R42: 100 Ω, Resistor_SMD:R_0603_1608Metric_Pad0.98x0.95mm_HandSolder, F.Cu at (97.0, 94.0)
- added R43: 100 Ω, Resistor_SMD:R_0603_1608Metric_Pad0.98x0.95mm_HandSolder, F.Cu at (156.2, 112.5)
- added R46: 100 Ω, Resistor_SMD:R_0603_1608Metric_Pad0.98x0.95mm_HandSolder, F.Cu at (162.1, 116.6)
- added R47: 100 Ω, Resistor_SMD:R_0603_1608Metric_Pad0.98x0.95mm_HandSolder, F.Cu at (158.4, 115.6)
- added R50: 100 Ω, Resistor_SMD:R_0603_1608Metric_Pad0.98x0.95mm_HandSolder, F.Cu at (128.5, 84.2)
- added R51: 33 Ω, Resistor_SMD:R_0603_1608Metric_Pad0.98x0.95mm_HandSolder, F.Cu at (184.9, 94.0)
- added R52: 100 Ω, Resistor_SMD:R_0603_1608Metric_Pad0.98x0.95mm_HandSolder, F.Cu at (128.5, 86.8)
- added R53: 33 Ω, Resistor_SMD:R_0603_1608Metric_Pad0.98x0.95mm_HandSolder, F.Cu at (184.9, 100.1)
- added R54: 33 Ω, Resistor_SMD:R_0603_1608Metric_Pad0.98x0.95mm_HandSolder, F.Cu at (184.9, 105.2)
- added R55: 33 Ω, Resistor_SMD:R_0603_1608Metric_Pad0.98x0.95mm_HandSolder, F.Cu at (184.9, 103.1)
- added R57: 33 Ω, Resistor_SMD:R_0603_1608Metric_Pad0.98x0.95mm_HandSolder, F.Cu at (184.9, 91.4)
- added R58: 33 Ω, Resistor_SMD:R_0603_1608Metric_Pad0.98x0.95mm_HandSolder, F.Cu at (181.4, 103.1)
- added R6: 100 Ω, Resistor_SMD:R_0603_1608Metric_Pad0.98x0.95mm_HandSolder, F.Cu at (128.5, 106.5)
- added R7: 100 Ω, Resistor_SMD:R_0603_1608Metric_Pad0.98x0.95mm_HandSolder, F.Cu at (132.1, 108.0)
- added R8: 100 Ω, Resistor_SMD:R_0603_1608Metric_Pad0.98x0.95mm_HandSolder, F.Cu at (250.8, 112.2)
- added R9: 100 Ω, Resistor_SMD:R_0603_1608Metric_Pad0.98x0.95mm_HandSolder, F.Cu at (246.0, 114.5)
- added SW2: PTS645VL58-2 LFS, Button_Switch_THT:SW_Tactile_SPST_Angled_PTS645Vx58-2LFS, F.Cu at (212.4, 73.9)
- added SW3: PTS645VL58-2 LFS, Button_Switch_THT:SW_Tactile_SPST_Angled_PTS645Vx58-2LFS, F.Cu at (262.2, 73.9)
- C3: value 10 µF -> 100 nF; footprint Capacitor_SMD:C_1206_3216Metric_Pad1.33x1.80mm_HandSolder -> Capacitor_SMD:C_0603_1608Metric_Pad1.08x0.95mm_HandSolder
- C5: value 100 nF -> 10 µF; footprint Capacitor_SMD:C_0603_1608Metric_Pad1.08x0.95mm_HandSolder -> Capacitor_SMD:C_1206_3216Metric_Pad1.33x1.80mm_HandSolder
- J1: value PJ-037A -> PJ-037AH
- R1: value 20 KΩ -> 5.1 KΩ
- SW1: footprint asl_footprints:switch_slide_DPDT -> asl_footprints:RA toggle
- U1: value R-78E5.0-1.0 -> TSR 3-2450N; footprint asl_footprints:Converter_DCDC_RECOM_R-78E-0.5_THT -> asl_footprints:Converter_DCDC_traco_3A
- U7, U8, U9: value TBD62083APG -> TBD62083AFNG,EL
- moved J5 103.5 mm to (113.8, 74.0), turned to 180 degrees
- moved C6 83.8 mm to (179.0, 97.5), turned to 180 degrees
- moved J4 51.8 mm to (226.0, 73.8), turned to 180 degrees
- moved R5 43.0 mm to (222.3, 80.8), turned to 0 degrees
- moved R4 41.7 mm to (229.0, 80.8), turned to 0 degrees
- moved R21 41.1 mm to (77.4, 111.0)
- moved R24 41.1 mm to (83.9, 90.8), turned to 90 degrees
- moved R26 41.1 mm to (82.3, 90.7), turned to 90 degrees
- moved R44 41.1 mm to (77.4, 104.2)
- moved R56 41.1 mm to (77.4, 97.5)
- moved R59 41.1 mm to (77.4, 90.8)
- moved S1 41.1 mm to (75.2, 113.6)
- moved S2 41.1 mm to (75.2, 106.7)
- moved S3 41.1 mm to (75.2, 99.8)
- moved S4 41.1 mm to (75.2, 92.9)
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- renumbered C2 to C4, D2 to D3, D3 to D4, D4 to D5, D5 to D6, J12 to J10, J13 to J11, J14 to J12, J15 to J13, J16 to J14, J17 to J15, J18 to J16, J4 to J2, J5 to J3, J6 to J4, J7 to J5, J9 to J7, J10 to J8, J11 to J9, R4 to R10, R6 to R17, R7 to R18, R8 to R19, R5 to R21, R9 to R24, R10 to R26, R12 to R37, R13 to R38, R2 to R4, R11 to R44, R14 to R45, R15 to R48, R16 to R49, R3 to R5, R17 to R56, R18 to R59, S3 to S1, S4 to S2, S5 to S3, S6 to S4, U13 to U11, U14 to U12, U15 to U13, U16 to U14, U17 to U15, U18 to U16, U19 to U17, U20 to U18, U21 to U19, U22 to U20
Connections:
- net Net-(S5-in1) renamed /BTN_B
- C3 pad 1: +5V -> +3.3V
- C5 pad 1: +3.3V -> +5V
- J2 pad 1: /1_C -> /BNC_1
- J3 pad 1: /6_C -> /BNC_2
- R1 pad 1: +12V -> +3.3V
- R1 pad 2: Net-(D1-A) -> Net-(D2-A)
- R21 pad 2: Net-(S3-in1) -> /BTN_D
- R44 pad 2: Net-(S4-in1) -> /BTN_C
- S1 pad 1: Net-(S3-in1) -> /BTN_D
- S1 pad 2: Net-(S3-in1) -> /BTN_D
- S2 pad 1: Net-(S4-in1) -> /BTN_C
- S2 pad 2: Net-(S4-in1) -> /BTN_C
- U10 pad 1: /D1 -> /D2
- U10 pad 3: /D2 -> /D1
- U10 pad 6: /D4 -> unconnected-(U10-IO4-Pad6)
- U2 pad 3: +5V -> VBUS
- U4 pad 22: /D1 -> Net-(U4-PA0)
- U4 pad 23: /D2 -> Net-(U4-PA1)
- U4 pad 24: /10_A -> Net-(U4-PA2(UART2_TX))
- U4 pad 25: /10_B -> Net-(U4-PA3(UART2_RX))
- U4 pad 28: /1_C -> Net-(U4-PA4(DAC1,I2S1_WS))
- U4 pad 29: /6_C -> Net-(U4-PA5(DAC2,I2S1_CK))
- U4 pad 30: /D3 -> Net-(U4-PA6(I2S1_SDI))
- U4 pad 31: /D4 -> Net-(U4-PA7(I2S1_SDO))
- U4 pad 35: /9_C -> unconnected-(U4-PB1-Pad35)
- U4 pad 37: /5_B -> Net-(U4-PE7(UART7_RX))
- U4 pad 38: /5_A -> Net-(U4-PE8(UART7_TX))
- U4 pad 39: /5_C -> Net-(U4-PE9)
- U4 pad 42: /8_C -> Net-(U4-PE12(SPI4_SCK))
- U4 pad 43: /8_B -> Net-(U4-PE13(SPI4_MISO))
- U4 pad 44: /8_A -> Net-(U4-PE14(SPI4_MOSI))
- U4 pad 46: /1_A -> Net-(U4-PB10(UART3_TX,_I2C2_SCL))
- U4 pad 47: /1_B -> Net-(U4-PB11(UART3_RX,_I2C2_SDA))
- U4 pad 51: /3_B -> Net-(U4-PB12(UART5_RX))
- U4 pad 52: /3_A -> Net-(U4-PB13(UART5_TX))
- U4 pad 53: /D8 -> Net-(U4-PB14)
- U4 pad 63: /4_A -> Net-(U4-PC6(UART6_TX))
- U4 pad 64: /4_B -> Net-(U4-PC7(UART6_RX))
- U4 pad 65: /4_C -> unconnected-(U4-PC8-Pad65)
- U4 pad 67: Net-(S3-in1) -> unconnected-(U4-PA8-Pad67)
- U4 pad 68: /9_A -> Net-(U4-PA9(UART1_TX))
- U4 pad 69: /9_B -> Net-(U4-PA10(UART1_RX))
- U4 pad 72: /D5 -> unconnected-(U4-PA13-Pad72)
- U4 pad 76: /D6 -> unconnected-(U4-PA14-Pad76)
- U4 pad 77: /D7 -> /BTN_D
- U4 pad 78: /2_A -> Net-(U4-PC10(UART4_TX))
- U4 pad 79: /2_B -> Net-(U4-PC11(UART4_RX))
- U4 pad 81: Net-(S4-in1) -> Net-(U4-PD0)
- U4 pad 82: /10_C -> Net-(U4-PD1)
- U4 pad 85: /BNC_1 -> /BTN_C
- U4 pad 86: /BNC_2 -> Net-(U4-PD5)
- U4 pad 89: /7_C -> Net-(U4-PB3(SPI3_SCK))
- U4 pad 90: /7_B -> Net-(U4-PB4(SPI3_MISO))
- U4 pad 91: /7_A -> Net-(U4-PB5(SPI3_MOSI))
- U4 pad 95: /6_A -> Net-(U4-PB8(I2C1_SCL,CAN1_RX))
- U4 pad 96: /6_B -> Net-(U4-PB9(I2C1_SDA,CAN1_TX))
Routing:
- net Net-(S3-in1): track 172.0 -> 0.00 mm, vias 4 -> 0
- net Net-(S4-in1): track 171.5 -> 0.00 mm, vias 4 -> 0
- net /BNC_1: track 181.7 -> 13.3 mm, vias 3 -> 0
- net /D8: track 163.1 -> 0.00 mm, vias 4 -> 0
- net /BTN_D: track 0.00 -> 148.0 mm, vias 0 -> 4
- net /D7: track 143.0 -> 0.00 mm, vias 3 -> 0
- net /D6: track 142.2 -> 0.00 mm, vias 3 -> 0
- net /BNC_2: track 152.9 -> 12.8 mm, vias 3 -> 0
- net /BTN_C: track 0.00 -> 136.1 mm, vias 0 -> 4
- net Net-(U4-PA3(UART2_RX)): track 0.00 -> 125.0 mm, vias 0 -> 6
- net /D5: track 145.8 -> 24.9 mm, vias 4 -> 1
- net /1_A: track 170.8 -> 56.9 mm, vias 1 -> 2
- net /10_B: track 124.8 -> 19.5 mm, vias 3 -> 1
- net /1_B: track 170.5 -> 66.6 mm, vias 2 -> 4
- net Net-(U4-PD1): track 0.00 -> 103.0 mm, vias 0 -> 4
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Other:
- board size 253 x 52 mm -> 215 x 60 mm
- board text added: "11_A"
- board text added: "11_B"
- board text added: "11_C"
- board text added: "11_PA"
- board text added: "11_PB"
- board text added: "DAC1"
- board text added: "DAC2"
- board text added: "v${REVISION} AUG 2026 AL"
- board text removed: "OFF"
- board text removed: "ON"

Commit message: pcb v0.9
Parts:
- removed JP1, JP2, JP3, JP4: M20-9990246, Connector_PinHeader_2.54mm:PinHeader_1x02_P2.54mm_Vertical
- removed the R32 at (177.8, 81.2)
- removed the R34 at (173.8, 79.8)
- removed the R36 at (114.0, 111.5)
- removed the R39 at (119.1, 112.5)
- added S5: CAS-D20TB, asl_footprints:CAS-D20TB, F.Cu at (66.2, 76.0)
- R11, R12, R13, R14, R15, R16, R20, R22, R23, R25, R27, R28, R29, R30, R31, R6, R7, R8, R9: value 100 Ω -> 33 Ω
- R32: renamed from R33; value 100 Ω -> 33 Ω
- R33: renamed from R35; value 100 Ω -> 33 Ω
- R36: renamed from R40; value 100 Ω -> 33 Ω
- R37: renamed from R41; value 100 Ω -> 33 Ω
- R38: renamed from R42; value 100 Ω -> 33 Ω
- R39: renamed from R43; value 100 Ω -> 33 Ω
- R42: renamed from R46; value 100 Ω -> 33 Ω
- R43: renamed from R47; value 100 Ω -> 33 Ω
- R46: renamed from R50; value 100 Ω -> 33 Ω
- R48: renamed from R52; value 100 Ω -> 33 Ω
- SW1: value 1825263-1 -> 100SP1T2B4M6QE
- TP1: footprint TestPoint:TestPoint_Keystone_5019_Miniature -> TestPoint:TestPoint_Plated_Hole_D2.0mm
- moved SW3 60.3 mm to (202.0, 73.9)
- moved R10 9.80 mm to (211.8, 82.5), turned to 180 degrees
- moved C4 7.15 mm to (244.5, 96.5)
- moved C5 7.02 mm to (253.5, 96.5)
- moved SW1 3.80 mm to (253.5, 87.0)
- moved R3 3.25 mm to (242.5, 89.5), turned to 90 degrees
- moved FID1 2.51 mm to (57.5, 75.8)
- moved TP1 2.24 mm to (224.8, 91.8), turned to 0 degrees
- moved U1 0.36 mm to (249.0, 100.5), turned to 180 degrees
- renumbered H3 to H2, H2 to H3, R37 to R34, R38 to R35, R44 to R40, R45 to R41, R48 to R44, R49 to R45, R51 to R47, R53 to R49, R54 to R50, R55 to R51, R56 to R52, R57 to R53, R58 to R54, R59 to R55
Connections:
- net /X_COM_A renamed /11_COM_A
- net /X_COM_B renamed /11_COM_B
- J6 pad 1: GND -> +12V
- J6 pad 2: +5V -> /11_PB
- J6 pad 3: +12V -> +5V
- J6 pad 4: /P1 -> /11_C
- J6 pad 5: /P2 -> /11_B
- J6 pad 6: /D1 -> /11_PA
- J6 pad 7: /D2 -> GND
- J6 pad 8: /D3 -> /11_A
- R14 pad 2: /D3 -> /11_C
- R46 pad 2: /D1 -> /11_A
- R48 pad 2: /D2 -> /11_B
- U10 pad 1: /D2 -> /11_B
- U10 pad 3: /D1 -> /11_A
- U10 pad 4: /D3 -> /11_C
- U10 pad 6: unconnected-(U10-IO4-Pad6) -> /D4
- U11 pad 4: /1_C -> /D5
- U11 pad 6: unconnected-(U11-IO4-Pad6) -> /1_C
- U4 pad 46: Net-(U4-PB10(UART3_TX,_I2C2_SCL)) -> /1_A
- U4 pad 47: Net-(U4-PB11(UART3_RX,_I2C2_SDA)) -> /1_B
- U4 pad 95: Net-(U4-PB8(I2C1_SCL,CAN1_RX)) -> /6_A
- U4 pad 96: Net-(U4-PB9(I2C1_SDA,CAN1_TX)) -> /6_B
- U7 pad 11: /P2 -> /11_PB
- U7 pad 12: /P1 -> /11_PA
Routing:
- net /1_A: track 56.9 -> 118.4 mm
- net /11_A: track 0.00 -> 60.2 mm, vias 0 -> 1
- net Net-(U4-PB10(UART3_TX,_I2C2_SCL)): track 59.9 -> 0.00 mm
- net /D5: track 24.9 -> 83.8 mm, vias 1 -> 3
- net /D2: track 57.7 -> 0.00 mm, vias 1 -> 0
- net /1_B: track 66.6 -> 124.2 mm
- net Net-(U4-PB11(UART3_RX,_I2C2_SDA)): track 55.8 -> 0.00 mm
- net /D1: track 54.0 -> 0.00 mm, vias 1 -> 0
- net /11_B: track 0.00 -> 53.8 mm, vias 0 -> 1
- net /BNC_2: track 12.8 -> 59.9 mm, vias 0 -> 1
- net /11_PA: track 0.00 -> 46.3 mm, vias 0 -> 1
- net /RST: track 119.9 -> 79.3 mm, vias 6 -> 5
- net /P2: track 38.3 -> 0.00 mm, vias 1 -> 0
- net /P1: track 38.1 -> 0.00 mm, vias 1 -> 0
- net /11_PB: track 0.00 -> 37.0 mm, vias 0 -> 1
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Other:
- board text added: "3.3V"
- board text added: "A"
- board text added: "B"
- board text added: "C"
- board text added: "D"
- board text added: "VBUS"
- board text added: "v${REVISION} OCT 2026 AL"
- board text removed: "D1"
- board text removed: "D10"
- board text removed: "D2"
- board text removed: "D3"
- board text removed: "D6"
- board text removed: "D7"
- board text removed: "D8"
- board text removed: "D9"
- board text removed: "DAC 1"
- board text removed: "DAC 2"
- board text removed: "P1"
- board text removed: "P2"
- board text removed: "USER"
- board text removed: "v${REVISION} AUG 2026 AL"
